Commit message: New urdf

File: src/seahawk_description/urdf/seahawk_description.urdf (robot description, URDF)
Before this commit: robot seahawk_description, 1 links, 0 joints
Links:
- link base_link: mass 6.91657871127401 -> 5.78614968628617; geometry collision mesh filename=package://RVIZ_Simplified_Module/meshes/base_link.STL; visual mesh filename=package://RVIZ_Simplified_Module/meshes/base_link.STL

Commit message: Changed stl file paths

File: src/seahawk_description/urdf/seahawk_description.urdf (robot description, URDF)
Before this commit: robot RVIZ_Simplified_Module, 1 links, 0 joints
Links:
- link base_link: geometry collision mesh filename=package://seahawk_description/meshes/base_link.STL; visual mesh filename=package://seahawk_description/meshes/base_link.STL

Commit message: Smaller file size for faster load time

File: src/seahawk_description/urdf/seahawk_description.urdf (robot description, URDF)
Before this commit: robot seahawk_description, 1 links, 0 joints
Links:
- link base_link: mass 5.78614968628617 -> 5.4230392489778
